File: Electronics/misa-pcb/Development_pcb/Development_pcb.kicad_sch (KiCad schematic)
At the start: 21 parts, among them J1 Pan-Servo, J2 Tilt-Servo, J3 cam-power, J4 laser-power, J5 SPEAKER, J6 TFT_display, J7 lidar-TOF, J8 USB_C_IN, Q1 PN2222A, U1 ESP32-S3-DEVKITC-1-N8R8, U2 MP3-TF-16P

Commit message: Add new components and testing scripts for MISA PCB project
- Created MP3-TF-16P symbol library for KiCad with detailed properties.
- Added HTML redirect page for SnapEDA import guide.
- Implemented MISA_Camera_Only_Test.py for camera functionality testing with face detection.
- Developed TEST_1_PanTilt.ino for pan/tilt servo control with safety limits.
- Created TEST_2_DFPlayer.ino for standalone DFPlayer testing with serial control.
- Added TEST_3_Laser.ino for laser module testing with safety reminders.
- Implemented TEST_4_LiDAR.ino for TF-Luna LIDAR distance measurement.
- Developed TEST_5_TFT.ino for TFT screen testing with color fill and border checks.
- Added yolov8n.pt model file for object detection.
- Introduced Doctor and Human classes in Java with constructors and methods for specialization and name handling.
Parts:
- added C6: 100µF 16v, Capacitor_THT:CP_Radial_D5.0mm_P2.50mm, symbol Device:C_Polarized_Small
- C1: renamed from C2; value 100nF -> 100nF 50v; footprint Capacitor_THT:C_Disc_D5.0mm_W2.5mm_P5.00mm -> Capacitor_THT:C_Disc_D5.0mm_W2.5mm_P2.50mm
- C2: renamed from C1; value 1000µF -> 1000µF 16v
- C3, C4: value 470µF -> 470µF 16v
- C5: value 100nF -> 100nF 50v; footprint Capacitor_THT:C_Disc_D5.0mm_W2.5mm_P5.00mm -> Capacitor_THT:C_Disc_D5.0mm_W2.5mm_P2.50mm
- D1: value SA5.0A -> SA6.0A
- F1: value Polyfuse -> MF-RG600; footprint Capacitor_THT:C_Disc_D5.0mm_W2.5mm_P5.00mm -> Fuse:Fuse_Bourns_MF-RG600
- J1, J2: footprint Connector_PinHeader_2.54mm:PinHeader_1x03_P2.54mm_Vertical -> Connector_JST:JST_XH_B3B-XH-A_1x03_P2.50mm_Vertical
- J7: footprint Connector_PinHeader_2.54mm:PinHeader_1x04_P2.54mm_Vertical -> Connector_JST:JST_XH_B4B-XH-A_1x04_P2.50mm_Vertical
- J8: footprint TerminalBlock_Phoenix:TerminalBlock_Phoenix_MKDS-3-2-5.08_1x02_P5.08mm_Horizontal -> TerminalBlock:TerminalBlock_Xinya_XY308-2.54-2P_1x02_P2.54mm_Horizontal
- R2: renamed from R4; value 1kΩ -> 220Ω
- renumbered R3 to R1
Connections:
- net TFT_MOSI is gone; now on net TFT_DC: J6.3 (Pin_3), U1.J1_5 (GPIO5)
- net TFT_SCK is gone; now on net TFT_CS: J6.2 (Pin_2), U1.J1_4 (GPIO4)
- net +3V3: now also J6.7 (Pin_7); no longer J6.8 (Pin_8)
- net +5V: now also J1.3 (Pin_3), J2.3 (Pin_3), C6.1; no longer J1.2 (Pin_2), J2.2 (Pin_2)
- net DF_RX: now also U1.J1_18 (GPIO12); no longer U1.J1_19 (GPIO13)
- net DF_TX: now also U1.J1_19 (GPIO13); no longer U1.J1_20 (GPIO14)
- net GND: now also J1.2 (Pin_2), J2.2 (Pin_2), J6.8 (Pin_8), C6.2; no longer J1.1 (Pin_1), J2.1 (Pin_1), J6.7 (Pin_7)
- net PAN_PWM: now also J1.1 (Pin_1), U1.J1_11 (GPIO18); no longer J1.3 (Pin_3), U1.J1_15 (GPIO9)
- net TFT_CS: no longer J6.6 (Pin_6), U1.J1_8 (GPIO15)
- net TFT_DC: no longer J6.4 (Pin_4), U1.J1_6 (GPIO6)
- net TFT_RST: now also J6.4 (Pin_4), U1.J1_6 (GPIO6); no longer J6.5 (Pin_5), U1.J1_7 (GPIO7)
- net TILT_PWM: now also J2.1 (Pin_1); no longer J2.3 (Pin_3)
- net DF_BUSY: now reaches U2.P$16 (BUSY)
- net DF_BUSY: now also U1.J1_20 (GPIO14)
- new net TFT_SCL: J6.6 (Pin_6), U1.J1_8 (GPIO15)
- new net TFT_SDA: J6.5 (Pin_5), U1.J1_7 (GPIO7)
- no-connect marks 35 -> 33
Other:
- moved on the sheet: C1, C2, C3, C4, D1, F1, J4, J5, J8, Q1, R2

Commit message: Refactor code structure for improved readability and maintainability
Parts:
- added C10, C14: 100µF 16v, Capacitor_THT:CP_Radial_D5.0mm_P2.50mm, symbol Device:C_Polarized_Small
- added C11, C7: 470µF 16v, Capacitor_THT:CP_Radial_D8.0mm_P3.50mm, symbol Device:C_Polarized_Small
- added C12, C13, C8, C9: 100nF 50v, Capacitor_THT:C_Disc_D5.0mm_W2.5mm_P2.50mm, symbol Device:C_Small
- C2: footprint Capacitor_THT:CP_Radial_D10.0mm_P5.00mm -> Capacitor_THT:CP_Radial_D12.5mm_P5.00mm
- R2: footprint Resistor_THT:R_Axial_DIN0207_L6.3mm_D2.5mm_P10.16mm_Horizontal -> Resistor_THT:R_Axial_DIN0207_L6.3mm_D2.5mm_P2.54mm_Vertical
Connections:
- net +3V3: now also C13.2, C14.1
- net +5V: now also C10.1, C11.1, C12.1, C9.1
- net GND: now also C10.2, C11.2, C12.2, C13.1, C14.2, C7.2, C8.1, C9.2
- net LASER_CTRL: now also U1.J1_17 (GPIO11); no longer U1.J3_5 (GPIO2)
- net at D2.1 (K), U1.J1_21 (5V0): now also C7.1, C8.2
Other:
- moved on the sheet: D2, J3, J5, J6

Commit message: Refactor code structure and remove redundant sections for improved readability and maintainability
Parts:
- added R3: 10kΩ, Resistor_THT:R_Axial_DIN0207_L6.3mm_D2.5mm_P2.54mm_Vertical, symbol Device:R_Small
- C10, C6: footprint Capacitor_THT:CP_Radial_D5.0mm_P2.50mm -> Capacitor_THT:CP_Radial_D6.3mm_P2.50mm
- R2: value 220Ω -> 100Ω
Connections:
- net +5V: now also J1.2 (Pin_2), J2.2 (Pin_2); no longer J1.3 (Pin_3), J2.3 (Pin_3)
- net GND: now also J1.3 (Pin_3), J2.3 (Pin_3), R3.1; no longer J1.2 (Pin_2), J2.2 (Pin_2)
- net at Q1.2 (B), R2.2: now also R3.2
Other:
- moved on the sheet: C1, C10, C11, C12, C13, C14, C2, C3, C4, C5, C6, C7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
